File: BreadBoardPower.sch (KiCad schematic (older format))
At the start: 15 parts, among them J1 USB_OTG, J2 Conn_01x02_Female, J3 Conn_02x04_Counter_Clockwise, J4 Conn_01x02_Male, J5 Conn_01x02_Male, SW1 SW_Push_SPDT, U1 AP1117-33

Commit message: commit
Parts:
- C1, C2, C3, C4, C5: symbol C_Small -> BreadBoardPower-rescue:C_Small
- D1: symbol LED -> BreadBoardPower-rescue:LED
- J1: symbol USB_OTG -> BreadBoardPower-rescue:USB_OTG
- J2: symbol Conn_01x02_Female -> BreadBoardPower-rescue:Conn_01x02_Female
- J3: symbol Conn_02x04_Counter_Clockwise -> BreadBoardPower-rescue:Conn_02x04_Counter_Clockwise
- J4, J5: symbol Conn_01x02_Male -> BreadBoardPower-rescue:Conn_01x02_Male
- L1: symbol Ferrite_Bead_Small -> BreadBoardPower-rescue:Ferrite_Bead_Small
- R1: symbol R_Small -> BreadBoardPower-rescue:R_Small
- SW1: symbol SW_Push_SPDT -> BreadBoardPower-rescue:SW_Push_SPDT
- U1: symbol AP1117-33 -> BreadBoardPower-rescue:AP1117-33
Changed lines of the file:
@@
-EESchema Schematic File Version 2
-LIBS:power
-LIBS:device
-LIBS:switches
-LIBS:relays
-LIBS:motors
-LIBS:transistors
-LIBS:conn
-LIBS:linear
-LIBS:regul
-LIBS:74xx
-LIBS:cmos4000
-LIBS:adc-dac
-LIBS:memory
-LIBS:xilinx
-LIBS:microcontrollers
-LIBS:dsp
-LIBS:microchip
-LIBS:analog_switches
-LIBS:motorola
-LIBS:texas
-LIBS:intel
-LIBS:audio
-LIBS:interface
-LIBS:digital-audio
-LIBS:philips
-LIBS:display
-LIBS:cypress
-LIBS:siliconi
-LIBS:opto
-LIBS:atmel
-LIBS:contrib
-LIBS:valves
+EESchema Schematic File Version 4
 LIBS:BreadBoardPower-cache
-EELAYER 25 0
+EELAYER 26 0
 EELAYER END
 $Descr A4 11693 8268
@@
 $EndDescr
 $Comp
-L USB_OTG J1
+L BreadBoardPower-rescue:USB_OTG J1
 U 1 1 5A20EF4F
 P 1650 1500
@@
 $EndComp
 $Comp
-L SW_Push_SPDT SW1
+L BreadBoardPower-rescue:SW_Push_SPDT SW1
 U 1 1 5A20F142
 P 3950 1300
@@
 $EndComp
 $Comp
-L C_Small C1
+L BreadBoardPower-rescue:C_Small C1
 U 1 1 5A2311DF
 P 4450 1100
@@
 $EndComp
 $Comp
-L C_Small C3
+L BreadBoardPower-rescue:C_Small C3
 U 1 1 5A2312DD
 P 5250 1100
@@
 Vout
 $Comp
-L AP1117-33 U1
+L BreadBoardPower-rescue:AP1117-33 U1
 U 1 1 5A28CCFF
 P 4850 1000
@@
 $EndComp
 $Comp
-L C_Small C4
+L BreadBoardPower-rescue:C_Small C4
 U 1 1 5A28D4D4
 P 2450 1600
@@
 $EndComp
 $Comp
-L C_Small C5
+L BreadBoardPower-rescue:C_Small C5
 U 1 1 5A28D512
 P 2850 1600
@@
 $EndComp
 $Comp
-L C_Small C2
+L BreadBoardPower-rescue:C_Small C2
 U 1 1 5A28D549
 P 2200 1600
@@
 $EndComp
 $Comp
-L Ferrite_Bead_Small L1
+L BreadBoardPower-rescue:Ferrite_Bead_Small L1
 U 1 1 5A28D845
 P 2650 1300
@@
 $EndComp
 $Comp
-L R_Small R1
+L BreadBoardPower-rescue:R_Small R1
 U 1 1 5A28DC08
 P 3300 1800
@@
 $EndComp
 $Comp
-L LED D1
+L BreadBoardPower-rescue:LED D1
 U 1 1 5A28DC47
 P 3300 1500
@@
 $EndComp
 Wire Wire Line
-	6100 1000 6100 1800
-Wire Wire Line
-	6100 1800 6400 1800
+	6100 1000 6100 1650
+Wire Wire Line
+	6100 1800 6250 1800
 Connection ~ 6100 1000
 Wire Wire Line
-	6000 1100 6400 1100
+	6000 1100 6250 1100
 Connection ~ 6000 1300
 Wire Wire Line
@@
 	4300 1200 4150 1200
 Wire Wire Line
-	1550 1900 6450 1900
-Wire Wire Line
-	2750 1300 3750 1300
-Wire Wire Line
-	4300 1000 4550 1000
+	1550 1900 1650 1900
+Wire Wire Line
+	2750 1300 2850 1300
+Wire Wire Line
+	4300 1000 4450 1000
 Wire Wire Line
 	4450 1200 4450 1300
-Connection ~ 4450 1300
 Connection ~ 4850 1300
 Wire Wire Line
@@
 Connection ~ 2850 1900
 Wire Wire Line
-	4450 1300 6000 1300
-Wire Wire Line
-	6000 1100 6000 1900
-$Comp
-L Conn_01x02_Male J4
+	4450 1300 4850 1300
+Wire Wire Line
+	6000 1100 6000 1300
+$Comp
+L BreadBoardPower-rescue:Conn_01x02_Male J4
 U 1 1 5A31F141
 P 6600 1100
@@
 $EndComp
 $Comp
-L Conn_01x02_Male J5
+L BreadBoardPower-rescue:Conn_01x02_Male J5
 U 1 1 5A31F2BD
 P 6600 1900
@@
 $EndComp
 $Comp
-L Conn_02x04_Counter_Clockwise J3
+L BreadBoardPower-rescue:Conn_02x04_Counter_Clockwise J3
 U 1 1 5A31F3A5
 P 7350 1400
@@
 $EndComp
 $Comp
-L Conn_01x02_Female J2
+L BreadBoardPower-rescue:Conn_01x02_Female J2
 U 1 1 5A28D865
 P 2100 2400
@@
 Connection ~ 6250 1800
 Wire Wire Line
-	1950 1300 2550 1300
+	1950 1300 2000 1300
 Wire Wire Line
 	2000 2200 2000 1300
@@
 	6250 1100 6250 1150
 Wire Wire Line
-	6250 1150 7450 1150
+	6250 1150 7250 1150
 Wire Wire Line
 	7450 1150 7450 1200
@@
 Connection ~ 6400 1000
 Wire Wire Line
-	7150 900  7150 1200
+	7150 900  7150 1000
 Connection ~ 7150 1000
 Wire Wire Line
 	6250 1800 6250 1750
 Wire Wire Line
-	6250 1750 7450 1750
+	6250 1750 7250 1750
 Wire Wire Line
 	7450 1750 7450 1700
@@
 	6450 1900 6450 2000
 Wire Wire Line
-	6400 2000 7350 2000
+	6400 2000 6450 2000
 Wire Wire Line
 	7350 2000 7350 1700
@@
 Connection ~ 7150 2000
 Wire Wire Line
-	5150 1000 6400 1000
+	5150 1000 5250 1000
 Wire Wire Line
 	6400 1000 6400 900
@@
 Connection ~ 6000 1900
 $Comp
-L GND #PWR?
+L BreadBoardPower-rescue:GND #PWR0101
 U 1 1 5A32C5F0
 P 3900 1900
-F 0 "#PWR?" H 3900 1650 50  0001 C CNN
+F 0 "#PWR0101" H 3900 1650 50  0001 C CNN
 F 1 "GND" H 3900 1750 50  0000 C CNN
 F 2 "" H 3900 1900 50  0001 C CNN
@@
 Connection ~ 3900 1900
 Connection ~ 1650 1900
+Wire Wire Line
+	6100 1000 6400 1000
+Wire Wire Line
+	6000 1300 6000 1900
+Wire Wire Line
+	4850 1300 5250 1300
+Wire Wire Line
+	5250 1300 6000 1300
+Wire Wire Line
+	2200 1300 2450 1300
+Wire Wire Line
+	2200 1900 2450 1900
+Wire Wire Line
+	2450 1900 2850 1900
+Wire Wire Line
+	2450 1300 2550 1300
+Wire Wire Line
+	2850 1300 3300 1300
+Wire Wire Line
+	2850 1900 3300 1900
+Wire Wire Line
+	6250 1100 6400 1100
+Wire Wire Line
+	6250 1800 6400 1800
+Wire Wire Line
+	2000 1300 2200 1300
+Wire Wire Line
+	2100 1900 2200 1900
+Wire Wire Line
+	5250 1000 6100 1000
+Wire Wire Line
+	4450 1000 4550 1000
+Wire Wire Line
+	6100 1650 6100 1800
+Wire Wire Line
+	3300 1900 3900 1900
+Wire Wire Line
+	3300 1300 3750 1300
+Wire Wire Line
+	7250 1150 7450 1150
+Wire Wire Line
+	7150 1000 7150 1200
+Wire Wire Line
+	7250 1750 7450 1750
+Wire Wire Line
+	6400 1900 6450 1900
+Wire Wire Line
+	7150 2000 7350 2000
+Wire Wire Line
+	6450 2000 7150 2000
+Wire Wire Line
+	6000 1900 6400 1900
+Wire Wire Line
+	3900 1900 6000 1900
+Wire Wire Line
+	1650 1900 2100 1900
 $EndSCHEMATC
